Commit message: add scaling option for the wheels

File: test/test_robot.urdf.xacro (robot description, xacro)
@@ -28,8 +28,8 @@
     <fdir1 value="0 1 0"/>
   </gazebo>
-  <xacro:mecanum_wheel name="front_right" side="1"  interface="hardware_interface/EffortJointInterface"/>
-  <xacro:mecanum_wheel name="front_left"  side="-1" interface="hardware_interface/EffortJointInterface"/>
-  <xacro:mecanum_wheel name="rear_right"  side="-1" interface="hardware_interface/EffortJointInterface"/>
-  <xacro:mecanum_wheel name="rear_left"   side="1"  interface="hardware_interface/EffortJointInterface"/>
+  <xacro:mecanum_wheel name="front_right" side="1"  interface="hardware_interface/EffortJointInterface" sf="1"/>
+  <xacro:mecanum_wheel name="front_left"  side="-1" interface="hardware_interface/EffortJointInterface" sf="1"/>
+  <xacro:mecanum_wheel name="rear_right"  side="-1" interface="hardware_interface/EffortJointInterface" sf="1"/>
+  <xacro:mecanum_wheel name="rear_left"   side="1"  interface="hardware_interface/EffortJointInterface" sf="1"/>
   <joint name="front_right_wheel_joint" type="continuous">
     <origin xyz="0.3 -0.25 -0.1" rpy="0 0 ${pi/2}" />

File: urdf/mecanum_wheel_macro.xacro (robot description, xacro)
@@ -3,7 +3,7 @@
   <xacro:include filename="$(find fuji_mecanum)/urdf/wheel.xacro" />
   <xacro:include filename="$(find fuji_mecanum)/urdf/rollers.xacro"  />
-  <xacro:macro name="mecanum_wheel" params="name side interface">
-    <xacro:wheel_link name="${name}" side="${side}" />
-    <xacro:rollers_link name="${name}" side="${side}" />
+  <xacro:macro name="mecanum_wheel" params="name side interface sf">
+    <xacro:wheel_link name="${name}" side="${side}" sf="${sf}"/>
+    <xacro:rollers_link name="${name}" side="${side}" sf="${sf}"/>
     <transmission name="${name}_wheel_trans">
       <type>transmission_interface/SimpleTransmission</type>

File: urdf/rollers.xacro (robot description, xacro)
@@ -1,13 +1,13 @@
 <?xml version="1.0" ?>
 <robot name="wheel" xmlns:xacro="http://www.ros.org/wiki/xacro">
-  <xacro:macro name="roller_origin" params="th side" >
+  <xacro:macro name="roller_origin" params="th side sf" >
     <xacro:if value="${side==1}">
-      <origin xyz="0 ${0.0895*cos(th)} ${0.0895*sin(th)}" rpy="${atan(-tan(th)*sqrt(2.0))} ${asin(cos(th)/sqrt(2.0))} ${atan(sin(th))}"/>
+      <origin xyz="0 ${sf*0.0895*cos(th)} ${sf*0.0895*sin(th)}" rpy="${atan(-tan(th)*sqrt(2.0))} ${asin(cos(th)/sqrt(2.0))} ${atan(sin(th))}"/>
     </xacro:if>
     <xacro:if value="${side==-1}">
-      <origin xyz="0 ${0.0895*cos(th)} ${0.0895*sin(th)}" rpy="${atan(-tan(th)*sqrt(2.0))} ${asin(-cos(th)/sqrt(2.0))} ${atan(-sin(th))}"/>
+      <origin xyz="0 ${sf*0.0895*cos(th)} ${sf*0.0895*sin(th)}" rpy="${atan(-tan(th)*sqrt(2.0))} ${asin(-cos(th)/sqrt(2.0))} ${atan(-sin(th))}"/>
     </xacro:if>
   </xacro:macro>
-  <xacro:macro name="roller_loop" params="name side num loop" >
+  <xacro:macro name="roller_loop" params="name side num loop sf" >
     <xacro:if value="${loop}">
       <link name="${name}_roller${loop}_link">
@@ -15,15 +15,15 @@
           <origin xyz="0 0 0" rpy="0 0 0" />
           <geometry>
-            <mesh filename="package://fuji_mecanum/mesh/visual/roller.dae" scale="1 1 1" />
+            <mesh filename="package://fuji_mecanum/mesh/visual/roller.dae" scale="${sf} ${sf} ${sf}" />
           </geometry>
         </visual>
         <collision>
           <geometry>
-            <mesh filename="package://fuji_mecanum/mesh/collision/roller.stl" scale="1 1 1" />
+            <mesh filename="package://fuji_mecanum/mesh/collision/roller.stl" scale="${sf} ${sf} ${sf}" />
           </geometry>
         </collision>
         <inertial>
           <origin xyz="0 0 0" />
-          <mass value="0.3" />
+          <mass value="${sf*0.3}" />
           <inertia ixx="0.00024000" ixy="0.0" ixz="0.0"
                   iyy="0.00076000" iyz="0.0"
@@ -32,5 +32,5 @@
       </link>
       <joint name="${name}_roller${loop}_joint" type="continuous">
-        <xacro:roller_origin th="${radians(360/num*(loop-1))}" side="${side}"/>
+        <xacro:roller_origin th="${radians(360/num*(loop-1))}" side="${side}" sf="${sf}"/>
         <axis xyz="1 0 0"/>
         <parent link="${name}_wheel_link" />
@@ -55,9 +55,9 @@
         <fdir1 value="0 1 0"/>
       </gazebo>
-      <xacro:roller_loop name="${name}" side="${side}" num="${num}" loop="${loop - 1}" />
+      <xacro:roller_loop name="${name}" side="${side}" num="${num}" loop="${loop - 1}" sf="${sf}" />
     </xacro:if>
   </xacro:macro>
-  <xacro:macro name="rollers_link" params="name side">
-    <xacro:roller_loop name="${name}" side="${side}" num="15" loop="15" />
+  <xacro:macro name="rollers_link" params="name side sf">
+    <xacro:roller_loop name="${name}" side="${side}" num="15" loop="15" sf="${sf}"/>
   </xacro:macro>
 </robot>

File: urdf/wheel.xacro (robot description, xacro)
@@ -1,20 +1,20 @@
 <?xml version="1.0" ?>
 <robot name="wheel" xmlns:xacro="http://www.ros.org/wiki/xacro">
-  <xacro:macro name="wheel_link" params="name side">
+  <xacro:macro name="wheel_link" params="name side sf">
     <link name="${name}_wheel_link">
       <visual>
         <origin xyz="0 0 0" rpy="0 0 0" />
         <geometry>
-          <mesh filename="package://fuji_mecanum/mesh/visual/wheel.dae" scale="${side} 1 1" />
+          <mesh filename="package://fuji_mecanum/mesh/visual/wheel.dae" scale="${(side)*(sf)} ${sf} ${sf}" />
         </geometry>
       </visual>
       <collision>
         <geometry>
-          <mesh filename="package://fuji_mecanum/mesh/collision/wheel.stl" scale="${side} 1 1" />
+          <mesh filename="package://fuji_mecanum/mesh/collision/wheel.stl" scale="${(side)*(sf)} ${sf} ${sf}" />
         </geometry>
       </collision>
       <inertial>
         <origin xyz="0 0 0" />
-        <mass value="2.0" />
+        <mass value="${sf*2.0}" />
         <inertia ixx="0.042025" ixy="0.0" ixz="0.0"
                 iyy="0.024279" iyz="0.0"
